Commit message: Last navigation version

File: noah_description/urdf/accurate_base_link.urdf.xacro (robot description, xacro)
@@ -304,4 +304,10 @@
 			<material>Gazebo/Blue</material>
 		</gazebo>
+		<joint name="imu_joint" type="fixed">
+			<parent link="front_link"/>
+			<child link="imu_link"/>
+			<origin xyz="0.0 0 0.068" rpy="0 0 0"/>
+		</joint>
+		<link name="imu_link"/>
 	</xacro:macro>
 </robot>
